File: examples/eyal/esp32/ESP32-eyal/ESP32-eyal.kicad_sch (KiCad schematic)
At the start: 30 parts, among them J1 Battery, J2 OW, J3 V1, J4 Serial, J5 VDD_I_SENSE, J6 BATT_I_SENSE, J7 ALT_V2, J8 ALT_V3, J9 Solar, Q1 2N7002W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

Commit message: Commit recent updates
Parts:
- added R12: 10K, Resistor_SMD:R_0805_2012Metric, symbol Device:R
- J4: footprint Connector_PinHeader_2.54mm:PinHeader_1x03_P2.54mm_Vertical -> Connector_PinHeader_2.54mm:PinHeader_1x05_P2.54mm_Vertical; symbol Connector_Generic:Conn_01x03 -> Connector_Generic:Conn_01x05
Connections:
- net EN: now also J4.5 (Pin_5), R12.2
- net PGM: now also J4.4 (Pin_4)
- net VDD: now also R12.1
Other:
- note added: "DTR"
- note added: "GND"
- note added: "RTS"
- note added: "RX"
- note added: "TX"
- moved on the sheet: Program1
