File: examples/eyal/esp32/ESP32-eyal/ESP32-eyal.kicad_pcb (KiCad board)
At the start: 2 copper layers, 99.7 x 99.7 mm, 173 parts, among them J1 Battery, J2 OW, J3 V1, J4 Serial, J5 VDD_I_SENSE, J6 BATT_I_SENSE, J7 ALT_V2, J8 ALT_V3, J9 Solar, Q1 2N7002W, Q2 DMP1045U, Q3 DMP1045U, Q4 DMP1045U, U1 RT9080-33, U2 ESP32-WROOM-32, U3 MCP73831

Commit message: Some adjustments in version 2
Parts:
- removed the REF** at (127.0, 50.2)
- removed the REF** at (145.4, 62.9)
- removed the REF** at (179.1, 97.2)
- removed the REF** at (167.0, 73.0)
- removed the REF** at (175.3, 60.4)
- removed the REF** at (179.1, 50.2)
- removed the REF** at (118.1, 50.2)
- removed the REF** at (181.6, 88.9)
- removed the REF** at (161.3, 80.6)
- removed the REF** at (150.2, 102.2)
- removed the REF** at (191.8, 120.0)
- removed the REF** at (105.4, 50.2)
- removed the REF** at (115.6, 60.3)
- removed the REF** at (153.7, 138.4)
- removed the REF** at (163.8, 138.4)
- removed the REF** at (128.9, 62.9)
- removed the REF** at (158.8, 124.5)
- removed the REF** at (191.8, 114.9)
- removed the REF** at (107.3, 62.9)
- removed the REF** at (149.9, 60.3)
- removed the REF** at (183.5, 62.9)
- removed the REF** at (108.0, 97.2)
- removed the REF** at (135.3, 52.7)
- removed the REF** at (143.5, 97.2)
- removed the REF** at (133.3, 60.3)
- removed the REF** at (153.7, 88.9)
- removed the REF** at (170.2, 50.2)
- removed the REF** at (161.2, 142.8)
- removed the REF** at (128.3, 88.9)
- removed the REF** at (152.4, 50.2)
- removed the REF** at (135.9, 88.9)
- removed the REF** at (137.2, 70.5)
- removed the REF** at (111.8, 70.5)
- removed the REF** at (133.3, 70.5)
- removed the REF** at (156.2, 142.9)
- removed the REF** at (146.1, 88.9)
- removed the REF** at (191.8, 128.9)
- removed the REF** at (183.5, 73.0)
- removed the REF** at (188.0, 70.5)
- removed the REF** at (182.9, 50.2)
- removed the REF** at (111.8, 60.3)
- removed the REF** at (175.3, 70.5)
- removed the REF** at (163.8, 114.9)
- removed the REF** at (181.6, 120.0)
- removed the REF** at (189.2, 124.5)
- removed the REF** at (158.8, 60.3)
- removed the REF** at (161.3, 128.9)
- removed the REF** at (187.3, 112.4)
- removed the REF** at (121.9, 50.2)
- removed the REF** at (174.6, 52.7)
- removed the REF** at (102.9, 60.3)
- removed the REF** at (120.7, 70.5)
- removed the REF** at (161.3, 50.2)
- removed the REF** at (124.5, 70.5)
- removed the REF** at (109.2, 50.2)
- removed the REF** at (107.3, 73.0)
- removed the REF** at (179.1, 142.9)
- removed the REF** at (125.7, 97.2)
- removed the REF** at (168.9, 124.5)
- removed the REF** at (125.7, 80.6)
- removed the REF** at (147.6, 106.6)
- removed the REF** at (115.6, 70.5)
- removed the REF** at (149.9, 70.5)
- removed the REF** at (156.2, 134.0)
- removed the REF** at (171.4, 120.0)
- removed the REF** at (120.7, 60.3)
- removed the REF** at (124.5, 60.3)
- removed the REF** at (161.3, 97.2)
- removed the REF** at (113.7, 52.7)
- removed the REF** at (187.3, 52.7)
- removed the REF** at (161.3, 120.0)
- removed the REF** at (177.8, 114.9)
- removed the REF** at (171.4, 128.9)
- removed the REF** at (150.2, 111.0)
- removed the REF** at (179.1, 84.5)
- removed the REF** at (159.4, 112.4)
- removed the REF** at (151.1, 128.9)
- removed the REF** at (162.6, 70.5)
- removed the REF** at (168.9, 114.9)
- removed the REF** at (171.4, 70.5)
- removed the REF** at (153.7, 70.5)
- removed the REF** at (161.2, 133.9)
- removed the REF** at (161.3, 93.3)
- removed the REF** at (173.4, 104.8)
- removed the REF** at (148.6, 50.2)
- removed the REF** at (163.8, 88.9)
- removed the REF** at (143.5, 84.5)
- removed the REF** at (173.4, 112.4)
- removed the REF** at (179.1, 70.5)
- removed the REF** at (108.0, 84.5)
- removed the REF** at (99.1, 60.3)
- removed the REF** at (191.8, 50.2)
- removed the REF** at (181.6, 128.9)
- removed the REF** at (167.0, 62.9)
- removed the REF** at (143.5, 80.6)
- removed the REF** at (130.8, 50.2)
- removed the REF** at (143.5, 93.3)
- removed the REF** at (141.0, 70.5)
- removed the REF** at (161.3, 84.5)
- removed the REF** at (139.7, 50.2)
- removed the REF** at (179.1, 93.3)
- removed the REF** at (188.0, 60.3)
- removed the REF** at (143.5, 50.2)
- removed the REF** at (110.5, 88.9)
- removed the REF** at (179.1, 134.0)
- removed the REF** at (141.0, 60.3)
- removed the REF** at (179.1, 124.5)
- removed the REF** at (187.3, 104.8)
- removed the REF** at (156.8, 52.7)
- removed the REF** at (125.7, 84.5)
- removed the REF** at (189.2, 138.4)
- removed the REF** at (108.0, 80.6)
- removed the REF** at (158.8, 70.5)
- removed the REF** at (102.9, 70.5)
- removed the REF** at (182.9, 114.9)
- removed the REF** at (145.4, 73.0)
- removed the REF** at (181.6, 138.4)
- removed the REF** at (128.9, 73.0)
- removed the REF** at (162.6, 60.3)
- removed the REF** at (171.4, 138.4)
- removed the REF** at (159.4, 104.8)
- removed the REF** at (99.1, 70.5)
- removed the REF** at (191.8, 60.3)
- removed the REF** at (171.4, 88.9)
- removed the REF** at (179.1, 60.3)
- removed the REF** at (189.2, 88.9)
- removed the REF** at (154.9, 114.9)
- removed the REF** at (179.1, 80.6)
- removed the REF** at (151.1, 120.0)
- removed the REF** at (118.1, 88.9)
- removed the REF** at (171.4, 60.3)
- removed the REF** at (191.8, 70.5)
- removed the REF** at (165.1, 50.2)
- removed the REF** at (108.0, 93.3)
- removed the REF** at (137.2, 60.4)
- removed the REF** at (148.6, 124.5)
- removed the REF** at (153.7, 60.3)
- removed the REF** at (125.7, 93.3)
- added C3: 4.7uF, Capacitor_SMD:C_0805_2012Metric_Pad1.18x1.45mm_HandSolder, F.Cu at (108.6, 139.1)
- added REF**: PinHeader_2x05_P2.54mm_Vertical, 0-Eyal:PinHeader_3x05_P2.54mm_Vertical, F.Cu at (144.8, 114.9)
- moved REF** 9.53 mm to (149.9, 102.2)
- moved REF** 9.53 mm to (149.9, 142.9)
- renumbered pgm to prog, rst to reset
Routing:
- net (no net): track 1054.5 -> 0.00 mm
- net VDD: track 106.5 -> 189.3 mm
- net unconnected-(U2-Pad27): track 0.00 -> 57.4 mm, vias 0 -> 1
- net unconnected-(U2-Pad23): track 0.00 -> 57.1 mm, vias 0 -> 1
- net unconnected-(U2-Pad28): track 0.00 -> 55.6 mm, vias 0 -> 1
- net unconnected-(U2-Pad30): track 0.00 -> 52.4 mm, vias 0 -> 1
- net unconnected-(U2-Pad31): track 0.00 -> 50.3 mm, vias 0 -> 1
- net GND: track 210.2 -> 234.0 mm
- net /SOLAR: track 9.26 -> 12.9 mm
Other:
- board text added: "15"
- board text added: "16"
- board text added: "17"
- board text added: "18"
- board text added: "19"
- board text added: "IO"
- board text added: "J10"
